File: kb60 - kicad/kb60.kicad_pcb (KiCad board)
At the start: 2 copper layers, 137 parts, among them U1 Raspberry_Pi_Pico

Commit message: started pcb design
placed keys in rough places
Parts:
- removed the D15 at (275.0, 72.7)
- removed the S15 at (285.8, 19.1)
- added SW1: RotaryEncoder_Switch, Rotary_Encoder:RotaryEncoder_Alps_EC12E-Switch_Vertical_H20mm, F.Cu at (727.7, 15.8)
- moved S43 509.9 mm to (724.4, 61.9)
- moved D1 509.4 mm to (766.9, 155.3)
- moved D2 509.4 mm to (766.9, 158.9)
- moved U1 509.4 mm to (773.6, 241.3)
- moved D10 509.4 mm to (763.1, 198.8)
- moved D11 509.4 mm to (763.1, 202.4)
- moved D12 509.4 mm to (763.1, 205.9)
- moved D13 509.4 mm to (763.1, 209.5)
- moved D14 509.4 mm to (763.1, 213.0)
- moved D16 509.4 mm to (773.9, 174.0)
- moved D17 509.4 mm to (773.9, 177.5)
- moved D18 509.4 mm to (773.9, 181.1)
- moved D19 509.4 mm to (773.9, 184.6)
- moved D20 509.4 mm to (773.9, 188.2)
- moved D21 509.4 mm to (773.9, 191.7)
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- renumbered D16 to D15, D17 to D16, D18 to D17, D19 to D18, D20 to D19, D21 to D20, D22 to D21, D23 to D22, D24 to D23, D25 to D24, D26 to D25, D27 to D26, D28 to D27, D29 to D28, D30 to D29, D31 to D30, D32 to D31, D33 to D32, D34 to D33, D35 to D34, D36 to D35, D37 to D36, D38 to D37, D39 to D38, D40 to D39, D41 to D40, D43 to D41, D44 to D42, D45 to D43, D46 to D44, D47 to D45, D48 to D46, D49 to D47, D50 to D48, D51 to D49, D52 to D50, D53 to D51, D54 to D52, D55 to D53, D56 to D54, D57 to D55, D58 to D56, D59 to D57, D60 to D58, D61 to D59, D62 to D60, D63 to D61, D67 to D62, D71 to D63, D72 to D64, D73 to D65, D74 to D66, D75 to D67, S16 to S15, S17 to S16, S18 to S17, S19 to S18, S20 to S19, S21 to S20, S22 to S21, S23 to S22, S24 to S23, S25 to S24, S26 to S25, S27 to S26, S28 to S27, S29 to S28, S30 to S29, S31 to S30, S32 to S31, S33 to S32, S34 to S33, S35 to S34, S36 to S35, S37 to S36, S38 to S37, S39 to S38, S40 to S39, S41 to S40, S43 to S41, S44 to S42, S45 to S43, S46 to S44, S47 to S45, S48 to S46, S49 to S47, S50 to S48, S51 to S49, S52 to S50, S53 to S51, S54 to S52, S55 to S53, S56 to S54, S57 to S55, S58 to S56, S59 to S57, S60 to S58, S61 to S59, S62 to S60, S63 to S61, S67 to S62, S71 to S63, S72 to S64, S73 to S65, S74 to S66, S75 to S67
Connections:
- U1 pad 26: unconnected-(U1-GPIO20-Pad26) -> Button
- U1 pad 27: unconnected-(U1-GPIO21-Pad27) -> Rotary A
- U1 pad 29: unconnected-(U1-GPIO22-Pad29) -> Rotary B
- U1 pad 3: unconnected-(U1-GND-Pad3) -> GND

Commit message: added rotary encoder to switch matrix
as it has a switch as well
also added my keyboard layout that i wanted as a guideline for pcb placement
Parts:
- added D68: Diode, ScottoKeebs_Components:Diode_DO-35, F.Cu at (781.0, 161.9)
- added G***: LOGO, kblayout:kbLayout2, F.Cu at (581.0, -23.8)
- moved S30 38.8 mm to (437.8, 95.2)
- moved S31 38.8 mm to (456.9, 95.2)
- moved S32 38.8 mm to (475.9, 95.2)
- moved S34 38.8 mm to (514.0, 95.2)
- moved S35 38.8 mm to (533.1, 95.2)
- moved S36 38.8 mm to (552.1, 95.2)
- moved S37 38.8 mm to (571.2, 95.2)
- moved S38 38.8 mm to (590.2, 95.2)
- moved S39 38.8 mm to (609.3, 95.2)
- moved S40 38.8 mm to (628.3, 95.2)
- moved S41 38.8 mm to (666.4, 95.2)
- moved S42 38.8 mm to (685.5, 95.2)
- moved S44 38.8 mm to (437.8, 114.3)
- moved S45 38.8 mm to (456.9, 114.3)
- moved S46 38.8 mm to (475.9, 114.3)
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Connections:
- SW1 pad S1: Button -> Net-(D68-A)
- SW1 pad S2: GND -> Column 14
- U1 pad 26: Button -> unconnected-(U1-GPIO20-Pad26)

Commit message: pcb layout mostly done and 3d models added
Parts:
- D1, D10, D11, D12, D13, D14, D15, D16, D17, D18, D19, D2, D20, D21, D22, D23, D24, D25, D26, D27, D28, D29, D3, D30, D31, D32, D33, D34, D35, D36, D37, D38, D39, D4, D40, D41, D42, D43, D44, D45, D46, D47, D48, D49, D5, D50, D51, D52, D53, D54, D55, D56, D57, D58, D59, D6, D60, D61, D62, D63, D64, D65, D66, D67, D68, D7, D8, D9, U1: moved to B.Cu
- moved D59 358.4 mm to (450.1, 137.2), turned to 90 degrees
- moved D44 349.9 mm to (450.1, 118.1), turned to 90 degrees
- moved D30 338.3 mm to (454.8, 99.1), turned to 90 degrees
- moved D60 335.2 mm to (473.9, 137.2), turned to 90 degrees
- moved D15 333.9 mm to (452.4, 80.0), turned to 90 degrees
- moved D1 332.9 mm to (447.7, 61.0), turned to 90 degrees
- moved D45 329.4 mm to (471.5, 118.1), turned to 90 degrees
- moved D2 315.7 mm to (466.7, 61.0), turned to 90 degrees
- moved D31 313.6 mm to (481.0, 99.1), turned to 90 degrees
- moved D61 312.2 mm to (497.7, 137.2), turned to 90 degrees
- moved D16 312.1 mm to (476.2, 80.0), turned to 90 degrees
- moved D46 309.0 mm to (492.9, 118.1), turned to 90 degrees
- moved D3 299.5 mm to (485.8, 61.0), turned to 90 degrees
- moved D32 296.2 mm to (500.1, 99.1), turned to 90 degrees
- moved D17 295.2 mm to (495.3, 80.0), turned to 90 degrees
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
Commit message: finished pcb placements
Parts:
- moved U1 328.6 mm to (419.1, 73.8)
Other:
- board outline added: 331 x 95.2 mm
Changed lines of the file:
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@@
 		)
 		(embedded_fonts no)
-		(model "${KICAD9_3DMODEL_DIR}/Rotary_Encoder.3dshapes/RotaryEncoder_Alps_EC12E-Switch_Vertical_H20mm.step"
+		(model "${KIPRJMOD}/libs/3dmodels/EC12 Encoder 10mm 3pin.stp"
 			(offset
-				(xyz 0 0 0)
+				(xyz 7.5 -2.5 0)
 			)
 			(scale
@@
 			)
 			(rotate
-				(xyz 0 0 0)
+				(xyz -0 -0 90)
 			)
 		)
@@
 		)
 		(embedded_fonts no)
-		(model "${SCOTTOKEEBS_KICAD}/3dmodels/ScottoKeebs_Components.3dshapes/Diode_DO-35.step"
+		(model "${KIPRJMOD}/libs/ScottoKicad/3dmodels/ScottoKeebs_Components.3dshapes/Diode_DO-35.step"
 			(offset
 				(xyz 0 0 0)
@@
 		)
 		(embedded_fonts no)
-		(model "${SCOTTOKEEBS_KICAD}/3dmodels/ScottoKeebs_Components.3dshapes/Diode_DO-35.step"
+		(model "${KIPRJMOD}/libs/ScottoKicad/3dmodels/ScottoKeebs_Components.3dshapes/Diode_DO-35.step"
 			(offset
 				(xyz 0 0 0)
@@
 		)
 		(embedded_fonts no)
-		(model "${SCOTTOKEEBS_KICAD}/3dmodels/ScottoKeebs_Components.3dshapes/Diode_DO-35.step"
+		(model "${KIPRJMOD}/libs/ScottoKicad/3dmodels/ScottoKeebs_Components.3dshapes/Diode_DO-35.step"
 			(offset
 				(xyz 0 0 0)
@@
 	(footprint "ScottoKeebs_MCU:Raspberry_Pi_Pico"
 		(layer "B.Cu")
-		(at 747.7125 73.81875 180)
+		(at 419.1 73.81875 180)
 		(property "Reference" "U1"
 			(at 0 32 0)
@@
 		)
 		(embedded_fonts no)
-		(model "${SCOTTOKEEBS_KICAD}/3dmodels/ScottoKeebs_Components.3dshapes/Diode_DO-35.step"
+		(model "${KIPRJMOD}/libs/ScottoKicad/3dmodels/ScottoKeebs_Components.3dshapes/Diode_DO-35.step"
 			(offset
 				(xyz 0 0 0)
@@
 		)
 		(embedded_fonts no)
-		(model "${SCOTTOKEEBS_KICAD}/3dmodels/ScottoKeebs_Components.3dshapes/Diode_DO-35.step"
+		(model "${KIPRJMOD}/libs/ScottoKicad/3dmodels/ScottoKeebs_Components.3dshapes/Diode_DO-35.step"
 			(offset
 				(xyz 0 0 0)
@@
 		)
 		(embedded_fonts no)
-		(model "${SCOTTOKEEBS_KICAD}/3dmodels/ScottoKeebs_Components.3dshapes/Diode_DO-35.step"
+		(model "${KIPRJMOD}/libs/ScottoKicad/3dmodels/ScottoKeebs_Components.3dshapes/Diode_DO-35.step"
 			(offset
 				(xyz 0 0 0)
@@
 		)
 		(embedded_fonts no)
-		(model "${SCOTTOKEEBS_KICAD}/3dmodels/ScottoKeebs_Components.3dshapes/Diode_DO-35.step"
+		(model "${KIPRJMOD}/libs/ScottoKicad/3dmodels/ScottoKeebs_Components.3dshapes/Diode_DO-35.step"
 			(offset
 				(xyz 0 0 0)
@@
 		)
 	)
+	(gr_rect
+		(start 404.8125 47.625)
+		(end 735.80625 142.875)
+		(stroke
+			(width 0.05)
+			(type default)
+		)
+		(fill no)
+		(layer "Edge.Cuts")
+	)
 	(embedded_fonts no)

Commit message: finished routing pcb
Parts:
- added G***: LOGO, kblayout:miku, F.Cu at (417.5, 127.0)
- added G***: LOGO, kblayout:chiikawa, B.Cu at (419.0, 121.5)
- moved D46 2.38 mm to (490.5, 118.1)
Routing:
- net Column 14: track 0.00 -> 363.0 mm, vias 0 -> 2
- net Row 4: track 0.00 -> 355.9 mm
- net Column 13: track 0.00 -> 353.7 mm, vias 0 -> 1
- net Rotary A: track 0.00 -> 340.8 mm
- net Row 1: track 0.00 -> 339.0 mm, vias 0 -> 2
- net Row 3: track 0.00 -> 336.3 mm
- net Row 0: track 0.00 -> 330.9 mm, vias 0 -> 2
- net Row 2: track 0.00 -> 328.4 mm, vias 0 -> 2
- net Column 12: track 0.00 -> 328.4 mm, vias 0 -> 4
- net Rotary B: track 0.00 -> 327.0 mm
- net Column 11: track 0.00 -> 305.1 mm, vias 0 -> 4
- net GND: track 0.00 -> 298.6 mm
- net Column 10: track 0.00 -> 297.3 mm, vias 0 -> 4
- net Column 9: track 0.00 -> 256.7 mm, vias 0 -> 1
- net Column 8: track 0.00 -> 231.5 mm, vias 0 -> 3
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Other:
- board size 331 x 95.2 mm -> 332 x 102 mm
- board text added: "hello there"
- board text added: "hiiii"
- board text added: "nothing here :("
- board text added: "shar <3"
- board text added: "space"
- board text added: "spin"

Commit message: added ground fill and prod files
Parts:
- removed the G*** at (581.0, -23.8)
Routing:
- added copper zone on B.Cu, net GND
- added copper zone on F.Cu, net GND

Commit message: made the pcb a lil smaller
and moved some components
Parts:
- moved S57 7.14 mm to (704.9, 114.3)
- moved D56 7.14 mm to (688.2, 118.1)
- moved D57 7.14 mm to (714.4, 118.1)
- moved S56 7.14 mm to (678.7, 114.3)
- moved S63 4.76 mm to (631.0, 133.3)
- moved S64 4.76 mm to (654.8, 133.3)
- moved D63 4.76 mm to (640.6, 137.2)
- moved D64 4.76 mm to (664.4, 137.2)
- moved D42 2.38 mm to (704.9, 99.1)
- moved D62 2.38 mm to (569.1, 137.2)
- moved S42 2.38 mm to (695.3, 95.2)
- moved S62 2.38 mm to (559.6, 133.3)
Routing:
- net Row 4: track 355.9 -> 360.6 mm
- net Column 10: track 297.3 -> 295.4 mm
- net Column 6: track 210.2 -> 211.2 mm
- net Net-(D42-A): track 7.51 -> 6.56 mm
- net Column 13: track 353.7 -> 353.4 mm, vias 1 -> 2
Other:
- board size 332 x 102 mm -> 332 x 99 mm

Commit message: upload kmk files
Parts:
- moved D42 2.38 mm to (702.5, 99.1)
- moved S42 2.38 mm to (692.9, 95.2)
Routing:
- net Column 13: track 353.4 -> 354.5 mm
Changed lines of the file:
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@@
 	(footprint "ScottoKeebs_MX:MX_PCB_1.00u"
 		(layer "F.Cu")
-		(at 695.325 95.25)
+		(at 692.94375 95.25)
 		(descr "MX keyswitch PCB Mount Keycap 1.00u")
 		(tags "MX Keyboard Keyswitch Switch PCB Cutout Keycap 1.00u")
@@
 	(footprint "ScottoKeebs_Components:Diode_DO-35"
 		(layer "B.Cu")
-		(at 704.85 99.06 90)
+		(at 702.46875 99.06 90)
 		(descr "Diode, DO-35_SOD27 series, Axial, Horizontal, pin pitch=7.62mm, , length*diameter=4*2mm^2, , http://www.diodes.com/_files/packages/DO-35.pdf")
 		(tags "Diode DO-35_SOD27 series Axial Horizontal pin pitch 7.62mm  length 4mm diameter 2mm")
@@
 	)
 	(segment
-		(start 704.85 99.06)
-		(end 671.5125 99.06)
+		(start 671.5125 99.06)
+		(end 702.46875 99.06)
 		(width 0.2)
 		(layer "F.Cu")
@@
 	)
 	(segment
+		(start 702.46875 99.06)
+		(end 733.425 99.06)
+		(width 0.2)
+		(layer "F.Cu")
+		(net 33)
+	)
+	(segment
 		(start 557.2125 99.06)
 		(end 576.2625 99.06)
@@
 	)
 	(segment
-		(start 733.425 99.06)
-		(end 704.85 99.06)
-		(width 0.2)
-		(layer "F.Cu")
-		(net 33)
-	)
-	(segment
 		(start 481.0125 99.06)
 		(end 500.0625 99.06)
@@
 	)
 	(segment
+		(start 696.2775 73.66)
+		(end 696.2775 85.56625)
+		(width 0.2)
+		(layer "B.Cu")
+		(net 82)
+	)
+	(segment
+		(start 689.5 101.5)
+		(end 691.515 101.5)
+		(width 0.2)
+		(layer "B.Cu")
+		(net 82)
+	)
+	(segment
+		(start 689.13375 101.13375)
+		(end 689.5 101.5)
+		(width 0.2)
+		(layer "B.Cu")
+		(net 82)
+	)
+	(segment
 		(start 437.5 94.270076)
 		(end 437.5 95.5)
@@
 	)
 	(segment
-		(start 437.5 95.5)
-		(end 439 97)
+		(start 688.5 101.5)
+		(end 689.5 101.5)
 		(width 0.2)
 		(layer "B.Cu")
@@
 	)
 	(segment
-		(start 683.5 101.5)
-		(end 691.515 101.5)
+		(start 437.5 95.5)
+		(end 439 97)
 		(width 0.2)
 		(layer "B.Cu")
@@
 	)
 	(segment
-		(start 680 98)
-		(end 683.5 101.5)
+		(start 683.5 101.5)
+		(end 688.5 101.5)
 		(width 0.2)
 		(layer "B.Cu")
@@
 	)
 	(segment
-		(start 696.2775 73.66)
-		(end 691.515 68.8975)
+		(start 696.2775 85.56625)
+		(end 689.13375 92.71)
 		(width 0.2)
 		(layer "B.Cu")
@@
 	)
 	(segment
-		(start 427.99 90.32875)
-		(end 433.558674 90.32875)
+		(start 689.13375 92.71)
+		(end 689.13375 101.13375)
 		(width 0.2)
 		(layer "B.Cu")
@@
 	)
 	(segment
-		(start 691.515 101.5)
-		(end 691.515 92.71)
+		(start 680 98)
+		(end 683.5 101.5)
 		(width 0.2)
 		(layer "B.Cu")
@@
 	)
 	(segment
-		(start 701.04 111.76)
-		(end 691.515 102.235)
+		(start 696.2775 73.66)
+		(end 691.515 68.8975)
 		(width 0.2)
 		(layer "B.Cu")
@@
 	)
 	(segment
-		(start 691.515 102.235)
-		(end 691.515 101.5)
+		(start 427.99 90.32875)
+		(end 433.558674 90.32875)
 		(width 0.2)
 		(layer "B.Cu")
@@
 	)
 	(segment
-		(start 701.04 130.81)
-		(end 701.04 111.76)
+		(start 701.04 111.76)
+		(end 691.515 102.235)
 		(width 0.2)
 		(layer "B.Cu")
@@
 	)
 	(segment
-		(start 691.515 92.71)
-		(end 696.2775 87.9475)
+		(start 691.515 102.235)
+		(end 691.515 101.5)
 		(width 0.2)
 		(layer "B.Cu")
@@
 	)
 	(segment
-		(start 696.2775 87.9475)
-		(end 696.2775 73.66)
+		(start 701.04 130.81)
+		(end 701.04 111.76)
 		(width 0.2)
 		(layer "B.Cu")
@@
 	)
 	(segment
-		(start 698.8175 90.17)
-		(end 700.0875 91.44)
+		(start 696.43625 90.17)
+		(end 697.70625 91.44)
 		(width 0.2)
 		(layer "F.Cu")
@@
 	)
 	(segment
-		(start 700.0875 91.44)
-		(end 704.85 91.44)
+		(start 697.70625 91.44)
+		(end 702.46875 91.44)
 		(width 0.2)
 		(layer "F.Cu")
