File: kb60 - kicad/kb60.kicad_pcb (KiCad board)
At the start: 2 copper layers, 332 x 99 mm, 139 parts, among them SW1 RotaryEncoder_Switch, U1 Raspberry_Pi_Pico

Commit message: add stabilizers to pcb
Parts:
- added REF**: Stabilizer_MX_6.25u, ScottoKeebs_Stabilizer:Stabilizer_MX_6.25u, F.Cu at (559.6, 133.3)
- added REF**: Stabilizer_MX_2.00u, ScottoKeebs_Stabilizer:Stabilizer_MX_2.00u, F.Cu at (695.3, 57.1)
- added REF**: Stabilizer_MX_2.00u, ScottoKeebs_Stabilizer:Stabilizer_MX_2.00u, F.Cu at (692.9, 95.2)
Routing:
- net GND: track 298.6 -> 300.6 mm
- net Rotary B: track 327.0 -> 329.0 mm
- net Rotary A: track 340.8 -> 342.0 mm
- net Column 14: track 363.0 -> 363.9 mm

Commit message: centered pcb in kicad
Parts:
- moved D41 363.3 mm to (311.0, 143.6)
- moved D65 363.3 mm to (334.8, 181.7)
- moved REF** 363.3 mm to (334.8, 101.6)
- moved S12 363.3 mm to (287.2, 101.6)
- moved S14 363.3 mm to (334.8, 101.6)
- moved S39 363.3 mm to (263.3, 139.7)
- moved D1 363.3 mm to (87.1, 105.5)
- moved D10 363.3 mm to (258.6, 105.5)
- moved D12 363.3 mm to (296.7, 105.5)
- moved D14 363.3 mm to (344.3, 105.5)
- moved D15 363.3 mm to (91.9, 124.5)
- moved D16 363.3 mm to (115.7, 124.5)
- moved D17 363.3 mm to (134.8, 124.5)
- moved D18 363.3 mm to (153.8, 124.5)
- moved D19 363.3 mm to (172.9, 124.5)
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
Commit message: removed 90 degree traces
was given feedback to as it is not best practice
Routing:
- net GND: track 300.6 -> 0.00 mm
- net Row 4: track 360.6 -> 385.1 mm
- net Column 2: track 147.4 -> 157.2 mm
- net Rotary B: track 329.0 -> 337.5 mm
- net Rotary A: track 342.0 -> 349.7 mm
- net Column 1: track 120.3 -> 116.2 mm
- net Column 13: track 354.5 -> 353.0 mm
- net Column 12: track 328.4 -> 327.8 mm
- net Row 2: vias 2 -> 1
- net Row 1: vias 2 -> 1
